File: DCdriver/DCdriver.sch (KiCad schematic (older format))
At the start: 8 parts, among them P1 CONTROL1, P2 35V, P3 GND, P4 5V, P5 OUT1, P6 CONTROL2, P7 OUT2, U1 L293D

Commit message: CleanUp
Changed lines of the file:
@@
 	5750 3700 6350 3700
 Wire Wire Line
-	6350 3700 6350 3900
-Wire Wire Line
-	6350 3900 6500 4000
-Wire Wire Line
-	6500 4100 5750 4000
+	6350 3700 6350 4000
 $Comp
 L CONN_01X01 P3
@@
 	1    0    0    -1
 $EndComp
+Wire Wire Line
+	5750 4000 6300 4000
+Wire Wire Line
+	6300 4000 6300 4100
+Wire Wire Line
+	6300 4100 6500 4100
+Wire Wire Line
+	6350 4000 6500 4000
 $EndSCHEMATC
