File: espDebug/espDebug.sch (KiCad schematic (older format))
At the start: 18 parts, among them P1 RAW, P2 3V3, P3 RX/TX, P4 CONN_01X09, P5 CONN_01X09, P6 CONN_01X02, P7 CONN_01X02, P8 3V3/GND, U1 SPX2920T-3.3, U2 ESP-201, U4 button

Commit message: Many uodates
Parts:
- removed P4, P5: CONN_01X09, Pin_Headers:Pin_Header_Straight_1x09, symbol CONN_01X09
- removed U1: SPX2920T-3.3, Power_Integrations:TO-220, symbol SPX2920T-3.3
- added CON1: BARREL_JACK, Connect:BARREL_JACK, symbol BARREL_JACK
- added D3: LED, LEDs:LED-3MM, symbol LED
- added P10: 3V3/GND, Pin_Headers:Pin_Header_Straight_2x03, symbol CONN_02X03
- added P4: ON/OFF, Pin_Headers:Pin_Header_Straight_2x01, symbol CONN_02X01
- added P5, P9: CONN_02X09, Pin_Headers:Pin_Header_Straight_2x09, symbol CONN_02X09
- added R8: 10k, Resistors_ThroughHole:Resistor_Horizontal_RM7mm, symbol R
- added R9: 1k, Resistors_ThroughHole:Resistor_Horizontal_RM7mm, symbol R
- added U1: BUTTON, bugs:button, symbol button
- added U3: AP1117-5, bugs:SMD-stab, symbol AP1117
- added U5: AP1117-3, bugs:SMD-stab, symbol AP1117
- added U6: button, bugs:button, symbol button
- P1: value RAW -> CONN_01X02
Connections:
- wire segments 73 -> 163
Other:
- moved on the sheet: D1, D2, P2, P3, P6, P7, P8, R1, R2, R3, R4, R5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
