File: espDebug/espDebug.kicad_pcb (KiCad board)
At the start: 2 copper layers, 14 parts, among them P1 RAW, P2 3V3, P3 RX/TX, U1 SPX2920T-3.3, U2 ESP-201, U3 ESP8266, U4 button

Commit message: Schematics updates
Parts:
- removed U3: ESP8266, bugs:esp8266
- added P4: CONN_01X09, Pin_Headers:Pin_Header_Straight_1x09, F.Cu at (129.5, 121.9)
- added P5: CONN_01X09, Pin_Headers:Pin_Header_Straight_1x09, F.Cu at (162.6, 101.6)
- added P6: CONN_01X02, Pin_Headers:Pin_Header_Straight_1x02, F.Cu at (124.5, 104.1)
- added P7: CONN_01X02, Pin_Headers:Pin_Header_Straight_1x02, F.Cu at (119.4, 104.1)
- added P8: 3V3/GND, Pin_Headers:Pin_Header_Straight_2x03, F.Cu at (144.8, 83.8)
- moved P1 30.5 mm to (162.6, 86.4)
- moved U1 15.3 mm to (157.5, 83.8), turned to 90 degrees
- moved D1 12.0 mm to (124.5, 127.0)
- moved D2 10.8 mm to (119.4, 124.5)
- moved R1 9.92 mm to (124.5, 119.4)
- moved R5 9.16 mm to (119.4, 116.8)
- moved R2 7.18 mm to (152.4, 101.6), turned to 270 degrees
- moved P2 6.84 mm to (144.8, 81.3)
- moved R4 5.24 mm to (149.9, 114.3), turned to 270 degrees
- moved R3 5.24 mm to (142.2, 109.2)
- moved U4 4.58 mm to (129.5, 88.9)
- moved P3 1.27 mm to (144.8, 94.0)
Connections:
- R1 pad 2: Net-(R1-Pad2) -> Net-(P6-Pad2)
- R5 pad 2: Net-(R5-Pad2) -> Net-(P7-Pad1)
- U2 pad 5: Net-(R5-Pad2) -> Net-(P4-Pad9)
- U2 pad 6: Net-(R1-Pad2) -> Net-(P4-Pad8)
- U4 pad 3: Net-(R5-Pad2) -> Net-(P4-Pad9)
Routing:
- net Net-(P3-Pad2): track 85.1 -> 5.08 mm
- net Net-(R5-Pad2): track 51.3 -> 0.00 mm
- net Net-(D1-Pad1): track 201.3 -> 152.6 mm
- net Net-(R1-Pad2): track 44.4 -> 0.00 mm
- net Net-(P3-Pad1): track 33.9 -> 5.08 mm
- net Net-(P4-Pad9): track 0.00 -> 28.6 mm
- net Net-(P4-Pad8): track 0.00 -> 10.2 mm
- net Net-(P5-Pad6): track 21.9 -> 12.7 mm
- net Net-(P5-Pad7): track 14.5 -> 20.3 mm
- net Net-(P5-Pad9): track 0.00 -> 5.08 mm
- net Net-(P5-Pad8): track 0.00 -> 5.08 mm
- net Net-(P5-Pad5): track 0.00 -> 5.08 mm
- net Net-(P5-Pad4): track 0.00 -> 5.08 mm
- net Net-(P5-Pad3): track 0.00 -> 5.08 mm
- net Net-(P5-Pad2): track 0.00 -> 5.08 mm
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
Commit message: Many uodates
Parts:
- added CON1: BARREL_JACK, Connect:BARREL_JACK, F.Cu at (116.8, 83.8)
- added D3: LED, LEDs:LED-3MM, F.Cu at (121.9, 73.7)
- added P10: 3V3/GND, Pin_Headers:Pin_Header_Straight_2x03, F.Cu at (161.3, 83.8)
- added P9: CONN_02X09, Pin_Headers:Pin_Header_Straight_2x09, F.Cu at (162.6, 101.6)
- added R8: 10k, Resistors_ThroughHole:Resistor_Horizontal_RM7mm, F.Cu at (144.8, 127.0)
- added R9: 1k, Resistors_ThroughHole:Resistor_Horizontal_RM7mm, F.Cu at (111.8, 73.7)
- added U3: AP1117-5, bugs:SMD-stab, F.Cu at (134.6, 81.3)
- added U5: AP1117-3, bugs:SMD-stab, F.Cu at (147.3, 78.7)
- added U6: button, bugs:button, F.Cu at (127.0, 129.5)
- P1: value RAW -> CONN_01X02
- P4: value CONN_01X09 -> ON/OFF; footprint Pin_Headers:Pin_Header_Straight_1x09 -> Pin_Headers:Pin_Header_Straight_2x01
- P5: value CONN_01X09 -> CONN_02X09; footprint Pin_Headers:Pin_Header_Straight_1x09 -> Pin_Headers:Pin_Header_Straight_2x09
- U1: value SPX2920T-3.3 -> BUTTON; footprint Power_Integrations:TO-220 -> bugs:button
- moved P4 52.1 mm to (141.0, 71.1), turned to 270 degrees
- moved P5 35.6 mm to (127.0, 101.6)
- moved U1 27.4 mm to (132.1, 73.7), turned to 270 degrees
- moved P1 13.4 mm to (156.8, 74.3), turned to 0 degrees
- moved P8 10.5 mm to (154.9, 86.4)
- moved P2 10.5 mm to (154.9, 83.8)
- moved D1 5.08 mm to (119.4, 127.0)
- moved D2 5.08 mm to (114.3, 124.5)
- moved P6 5.08 mm to (119.4, 104.1)
- moved P7 5.08 mm to (114.3, 104.1)
- moved R1 5.08 mm to (119.4, 119.4)
- moved R5 5.08 mm to (114.3, 116.8)
- moved U4 2.54 mm to (129.5, 91.4)
Connections:
- D1 pad 1: Net-(D1-Pad1) -> Net-(CON1-Pad2)
- D2 pad 1: Net-(D1-Pad1) -> Net-(CON1-Pad2)
- P1 pad 2: Net-(D1-Pad1) -> Net-(CON1-Pad2)
- P2 pad 2: Net-(D1-Pad1) -> Net-(CON1-Pad2)
- P4 pad 2: Net-(P4-Pad2) -> Net-(D3-Pad2)
- P5 pad 2: Net-(P5-Pad2) -> Net-(P5-Pad1)
- P5 pad 4: Net-(P5-Pad4) -> Net-(P5-Pad3)
- P5 pad 6: Net-(P5-Pad6) -> Net-(P5-Pad5)
- P5 pad 8: Net-(P5-Pad8) -> Net-(P5-Pad7)
- P5 pad 9: Net-(P5-Pad9) -> Net-(P5-Pad10)
- P6 pad 1: Net-(P4-Pad8) -> Net-(P5-Pad3)
- P7 pad 2: Net-(P4-Pad9) -> Net-(P5-Pad1)
- P8 pad 2: Net-(D1-Pad1) -> Net-(CON1-Pad2)
- P8 pad 4: Net-(D1-Pad1) -> Net-(CON1-Pad2)
- P8 pad 6: Net-(D1-Pad1) -> Net-(CON1-Pad2)
- R2 pad 1: Net-(P5-Pad1) -> Net-(P9-Pad1)
- R2 pad 2: Net-(D1-Pad1) -> Net-(CON1-Pad2)
- R3 pad 2: Net-(P5-Pad7) -> Net-(P9-Pad13)
- R4 pad 1: Net-(P5-Pad6) -> Net-(P9-Pad11)
- U1 pad 2: Net-(D1-Pad1) -> Net-(P4-Pad1)
- U1 pad 3: Net-(P2-Pad1) -> Net-(U1-Pad3)
- U2 pad 10: Net-(P4-Pad4) -> Net-(P5-Pad11)
- U2 pad 11: Net-(P4-Pad3) -> Net-(P5-Pad13)
- U2 pad 12: Net-(P4-Pad2) -> Net-(P5-Pad15)
- U2 pad 13: Net-(P4-Pad1) -> Net-(P5-Pad17)
- U2 pad 18: Net-(P5-Pad9) -> Net-(P9-Pad17)
- U2 pad 19: Net-(P5-Pad8) -> Net-(P9-Pad15)
- U2 pad 20: Net-(P5-Pad7) -> Net-(P9-Pad13)
- U2 pad 21: Net-(P5-Pad6) -> Net-(P9-Pad11)
- U2 pad 22: Net-(P5-Pad5) -> Net-(P9-Pad10)
- U2 pad 23: Net-(P5-Pad4) -> Net-(P9-Pad7)
- U2 pad 24: Net-(P5-Pad3) -> Net-(P9-Pad5)
- U2 pad 25: Net-(P5-Pad2) -> Net-(P9-Pad3)
- U2 pad 26: Net-(P5-Pad1) -> Net-(P9-Pad1)
- U2 pad 4: Net-(D1-Pad1) -> Net-(CON1-Pad2)
- U2 pad 5: Net-(P4-Pad9) -> Net-(P5-Pad1)
- U2 pad 6: Net-(P4-Pad8) -> Net-(P5-Pad3)
- U2 pad 7: Net-(P4-Pad7) -> Net-(P5-Pad5)
- U2 pad 8: Net-(P4-Pad6) -> Net-(P5-Pad7)
- U2 pad 9: Net-(P4-Pad5) -> Net-(P5-Pad10)
- U4 pad 1: Net-(U4-Pad1) -> Net-(CON1-Pad2)
- U4 pad 2: Net-(D1-Pad1) -> Net-(P5-Pad1)
- U4 pad 3: Net-(P4-Pad9) -> Net-(U4-Pad3)
Routing:
- net Net-(CON1-Pad2): track 0.00 -> 197.9 mm
- net Net-(D1-Pad1): track 152.6 -> 0.00 mm
- net Net-(CON1-Pad1): track 5.08 -> 66.1 mm
- net Net-(P5-Pad17): track 0.00 -> 37.7 mm
- net Net-(P4-Pad9): track 28.6 -> 0.00 mm
- net Net-(D3-Pad2): track 0.00 -> 23.2 mm
- net Net-(P5-Pad1): track 10.2 -> 33.0 mm
- net Net-(P9-Pad13): track 0.00 -> 22.9 mm
- net Net-(P9-Pad11): track 0.00 -> 15.2 mm
- net Net-(P9-Pad1): track 0.00 -> 12.7 mm
- net Net-(P5-Pad7): track 20.3 -> 7.62 mm
- net Net-(P5-Pad6): track 12.7 -> 0.00 mm
- net Net-(P4-Pad8): track 10.2 -> 0.00 mm
- net Net-(P5-Pad3): track 5.08 -> 15.2 mm
- net Net-(P9-Pad7): track 0.00 -> 7.62 mm
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