File: lineSensor/lineSensor.sch (KiCad schematic (older format))
At the start: 36 parts, among them P1 CONN_01X01, P10 CONN_01X01, P11 CONN_01X01, P12 CONN_01X01, P13 CONN_01X01, P14 CONN_01X01, P15 CONN_01X01, P2 CONN_01X01, P3 CONN_01X01, P4 CONN_01X01, P5 CONN_01X01, P6 CONN_01X01, P7 CONN_01X01, P8 CONN_01X01, P9 CONN_01X01

Commit message: CleanUp
Parts:
- removed P14, P15: CONN_01X01, Pin_Headers:Pin_Header_Straight_1x01, symbol CONN_01X01
- removed R11: 8k2, w_pth_resistors:rc05_vert, symbol R
Changed lines of the file:
@@
 	3300 2800 3750 2800
 Connection ~ 3550 2800
-$Comp
-L CONN_01X01 P15
-U 1 1 5728B887
-P 2650 4050
-F 0 "P15" H 2650 4150 50  0000 C CNN
-F 1 "CONN_01X01" V 2750 4050 50  0000 C CNN
-F 2 "Pin_Headers:Pin_Header_Straight_1x01" H 2650 4050 50  0001 C CNN
-F 3 "" H 2650 4050 50  0000 C CNN
-	1    2650 4050
-	-1   0    0    1
-$EndComp
-$Comp
-L R R11
-U 1 1 5728B949
-P 2850 3800
-F 0 "R11" V 2930 3800 50  0000 C CNN
-F 1 "8k2" V 2850 3800 50  0000 C CNN
-F 2 "w_pth_resistors:rc05_vert" V 2780 3800 50  0001 C CNN
-F 3 "" H 2850 3800 50  0000 C CNN
-	1    2850 3800
-	1    0    0    -1
-$EndComp
-$Comp
-L CONN_01X01 P14
-U 1 1 5728BAAE
-P 2650 3550
-F 0 "P14" H 2650 3650 50  0000 C CNN
-F 1 "CONN_01X01" V 2750 3550 50  0000 C CNN
-F 2 "Pin_Headers:Pin_Header_Straight_1x01" H 2650 3550 50  0001 C CNN
-F 3 "" H 2650 3550 50  0000 C CNN
-	1    2650 3550
-	-1   0    0    1
-$EndComp
-Wire Wire Line
-	2850 3650 2850 3550
-Wire Wire Line
-	2850 3950 2850 4050
 $EndSCHEMATC

Commit message: Components for BUG
Parts:
- P1, P10, P12, P13: value CONN_01X01 -> 5V
- P11, P2, P8, P9: value CONN_01X01 -> GND
Changed lines of the file:
@@
 P 4100 3550
 F 0 "P1" V 4100 3650 50  0000 C CNN
-F 1 "CONN_01X01" V 4200 3550 50  0000 C CNN
+F 1 "5V" V 4200 3550 50  0000 C CNN
 F 2 "Pin_Headers:Pin_Header_Straight_1x01" H 4100 3550 50  0001 C CNN
 F 3 "" H 4100 3550 50  0000 C CNN
@@
 P 4100 4350
 F 0 "P2" H 4100 4450 50  0000 C CNN
-F 1 "CONN_01X01" V 4200 4350 50  0000 C CNN
+F 1 "GND" V 4200 4350 50  0000 C CNN
 F 2 "Pin_Headers:Pin_Header_Straight_1x01" H 4100 4350 50  0001 C CNN
 F 3 "" H 4100 4350 50  0000 C CNN
@@
 P 4200 2600
 F 0 "P10" V 4200 2700 50  0000 C CNN
-F 1 "CONN_01X01" V 4300 2600 50  0000 C CNN
+F 1 "5V" V 4300 2600 50  0000 C CNN
 F 2 "Pin_Headers:Pin_Header_Straight_1x01" H 4200 2600 50  0001 C CNN
 F 3 "" H 4200 2600 50  0000 C CNN
@@
 P 3750 2600
 F 0 "P8" V 3750 2700 50  0000 C CNN
-F 1 "CONN_01X01" V 3850 2600 50  0000 C CNN
+F 1 "GND" V 3850 2600 50  0000 C CNN
 F 2 "Pin_Headers:Pin_Header_Straight_1x01" H 3750 2600 50  0001 C CNN
 F 3 "" H 3750 2600 50  0000 C CNN
@@
 P 3550 2600
 F 0 "P11" V 3550 2700 50  0000 C CNN
-F 1 "CONN_01X01" V 3650 2600 50  0000 C CNN
+F 1 "GND" V 3650 2600 50  0000 C CNN
 F 2 "Pin_Headers:Pin_Header_Straight_1x01" H 3550 2600 50  0001 C CNN
 F 3 "" H 3550 2600 50  0000 C CNN
@@
 P 3300 2600
 F 0 "P9" V 3300 2700 50  0000 C CNN
-F 1 "CONN_01X01" V 3400 2600 50  0000 C CNN
+F 1 "GND" V 3400 2600 50  0000 C CNN
 F 2 "Pin_Headers:Pin_Header_Straight_1x01" H 3300 2600 50  0001 C CNN
 F 3 "" H 3300 2600 50  0000 C CNN
@@
 P 4350 2600
 F 0 "P12" V 4350 2700 50  0000 C CNN
-F 1 "CONN_01X01" V 4450 2600 50  0000 C CNN
+F 1 "5V" V 4450 2600 50  0000 C CNN
 F 2 "Pin_Headers:Pin_Header_Straight_1x01" H 4350 2600 50  0001 C CNN
 F 3 "" H 4350 2600 50  0000 C CNN
@@
 P 4550 2600
 F 0 "P13" V 4550 2700 50  0000 C CNN
-F 1 "CONN_01X01" V 4650 2600 50  0000 C CNN
+F 1 "5V" V 4650 2600 50  0000 C CNN
 F 2 "Pin_Headers:Pin_Header_Straight_1x01" H 4550 2600 50  0001 C CNN
 F 3 "" H 4550 2600 50  0000 C CNN
