File: BUG/SonarAndLineFollowerAndIR/SonarAndLineFollowerAndIRR.sch (KiCad schematic (older format))
At the start: 24 parts, among them J1 RJ12, P2 Sonar, P3 CONN_01X03, U1 Arduino_Mini

Commit message: Schematics updates
Parts:
- added P1: IRT, Pin_Headers:Pin_Header_Straight_1x02, symbol CONN_01X02
- added P4: CONN_01X03, Pin_Headers:Pin_Header_Straight_1x03, symbol CONN_01X03
- added P5, P6: under, Pin_Headers:Pin_Header_Straight_1x01, symbol CONN_01X01
- added R11: R, Resistors_ThroughHole:Resistor_Horizontal_RM7mm, symbol R
- added R12, R13, R14, R15: 0, Resistors_SMD:R_1206, symbol R
- P3: value CONN_01X03 -> IRR
- R1, R10, R2, R3, R4, R5, R6, R7, R8, R9: footprint Resistors_ThroughHole:Resistor_Horizontal_RM15mm -> Resistors_ThroughHole:Resistor_Horizontal_RM7mm
Connections:
- net at D1.2 (A), D10.2 (A), D2.2 (A)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: now also R13.1, R14.2; no longer P2.1 (P1), P3.3 (P3), U1.10 (VCC)
- net at D2.1 (K), R2.1: now also U1.14 (A0); no longer U1.23 (A4)
- net at D4.1 (K), R4.1: now also U1.12 (A2); no longer U1.11 (A3)
- net at D8.1 (K), R8.1: now also U1.11 (A3); no longer U1.12 (A2)
- net at D10.1 (K), R10.1: now also R15.2; no longer U1.14 (A0)
- net at P2.4 (P4), P3.2 (P2), R10.2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: now also J1.2, R12.2; no longer J1.6, R1.2, R2.2, R3.2, R4.2, R5.2
- net at P3.1 (P1): now also U1.28 (5); no longer U1.30 (3)
- net at U1.15 (13): now also J1.3
- net at U1.16 (12): now also J1.5
- net at U1.17 (11): now also J1.6
- net at U1.18 (10): now also P4.3 (P3)
- net at U1.32 (GND): now also P1.1 (P1)
- net at U1.33 (RST): no longer J1.4
- net at U1.34 (RXI): no longer J1.2
- net at U1.35 (TXO): no longer J1.1
- net at U1.7 (RAW): now also J1.1; no longer J1.5
- net at U1.9 (RST): now also P4.1 (P1)
- new net: R1.2, R12.1, R2.2, R3.2, R4.2, R5.2
- new net: P2.1 (P1), P3.3 (P3), R14.1
- new net: P5.1 (P1), R13.2, U1.10 (VCC)
- new net: P6.1 (P1), R15.1, U1.23 (A4)
- new net: R11.1, U1.30 (3)
- new net: J1.4, P4.2 (P2)
- new net: P1.2 (P2), R11.2
Other:
- moved on the sheet: J1, P3
