File: BUG/SonarAndLineFollowerAndIR/SonarAndLineFollowerAndIRR.kicad_pcb (KiCad board)
At the start: 2 copper layers, 33 parts, among them J1 RJ12, P1 IRT, P2 Sonar, P3 IRR, P4 CONN_01X03, P5 under, P6 under, U1 Arduino_Mini

Commit message: Many uodates
Routing:
- net Net-(D6-Pad1): track 23.1 -> 26.0 mm
Changed lines of the file:
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@@
     (visible_elements FFFFFF7F)
     (pcbplotparams
-      (layerselection 0x00000_80000000)
+      (layerselection 0x00000_80000001)
       (usegerberextensions false)
       (excludeedgelayer true)
@@
   (segment (start 134.62 111.76) (end 137.16 111.76) (width 0.4) (layer B.Cu) (net 5))
   (segment (start 147.32 114.3) (end 147.32 116.84) (width 0.4) (layer B.Cu) (net 6))
-  (segment (start 147.32 124.46) (end 149.225 124.46) (width 0.4) (layer F.Cu) (net 7))
-  (segment (start 154.94 130.175) (end 154.94 137.16) (width 0.4) (layer F.Cu) (net 7))
-  (segment (start 149.225 124.46) (end 154.94 130.175) (width 0.4) (layer F.Cu) (net 7))
+  (segment (start 142.24 127) (end 149.86 127) (width 0.4) (layer F.Cu) (net 7))
+  (segment (start 154.94 132.08) (end 154.94 137.16) (width 0.4) (layer F.Cu) (net 7))
+  (segment (start 149.86 127) (end 154.94 132.08) (width 0.4) (layer F.Cu) (net 7))
   (segment (start 147.32 124.46) (end 144.78 124.46) (width 0.4) (layer B.Cu) (net 7))
   (segment (start 144.78 124.46) (end 142.24 127) (width 0.4) (layer B.Cu) (net 7))
