File: BUG/SonarAndLineFollowerAndIRR/SonarAndLineFollowerAndIRR.kicad_pcb (KiCad board)
At the start: 2 copper layers, 24 parts, among them J1 RJ12, P2 Sonar, P3 CONN_01X03, U1 Arduino_Mini

Commit message: Schematics updates
Parts:
- J1: footprint Connect:RJ12_E -> bugs:RJ12_Client
Connections:
- U1 pad 33: Net-(U1-Pad33) -> Net-(J1-Pad4)
- U1 pad 34: Net-(J1-Pad1) -> Net-(J1-Pad2)
- U1 pad 35: Net-(J1-Pad2) -> Net-(J1-Pad1)
Routing:
- net Net-(J1-Pad2): track 59.5 -> 23.7 mm
- net Net-(J1-Pad4): track 9.25 -> 42.9 mm
- net Net-(J1-Pad1): track 43.8 -> 14.4 mm
- net Net-(J1-Pad5): track 28.0 -> 12.7 mm
Other:
- net class Default: trace_width 0.75 -> 0.4
