File: BUG/WheelsAndIRT/WheelsAndIRT.kicad_pcb (KiCad board)
At the start: 2 copper layers, 8 parts, among them J1 RJ12, P1 CONN_01X05, P2 CONN_01X05, P3 CONN_01X01, P4 IRT, U1 uln2803A, U2 Arduino_Mini

Commit message: Update WheelsAndIRT
Parts:
- J1: footprint Connect:RJ12_E -> bugs:RJ12_Client
- moved P4 34.2 mm to (172.7, 85.1), turned to 270 degrees
- moved R1 23.9 mm to (175.3, 90.2), turned to 270 degrees
- moved P2 7.73 mm to (148.6, 109.2)
- moved P1 6.35 mm to (148.6, 127.0)
- moved P3 2.69 mm to (154.3, 95.9)
- moved U1 1.27 mm to (161.3, 127.0)
Connections:
- U2 pad 18: Net-(P4-Pad2) -> Net-(U1-Pad7)
- U2 pad 30: Net-(U1-Pad7) -> Net-(P4-Pad2)
- U2 pad 34: Net-(J1-Pad1) -> Net-(J1-Pad2)
- U2 pad 35: Net-(J1-Pad2) -> Net-(J1-Pad1)
Routing:
- net Net-(U1-Pad7): track 5.08 -> 43.0 mm
- net Net-(J1-Pad5): track 131.9 -> 113.2 mm
- net Net-(P4-Pad2): track 11.2 -> 29.5 mm
- net Net-(J1-Pad2): track 16.3 -> 34.1 mm
- net Net-(J1-Pad1): track 23.2 -> 39.0 mm
- net Net-(P2-Pad4): track 5.08 -> 11.2 mm
- net Net-(P2-Pad3): track 5.08 -> 10.5 mm
- net Net-(P2-Pad2): track 5.08 -> 10.5 mm
- net Net-(P1-Pad4): track 10.2 -> 5.08 mm
- net Net-(P1-Pad3): track 10.2 -> 5.08 mm
- net Net-(P1-Pad2): track 10.2 -> 5.08 mm
- net Net-(P1-Pad1): track 10.2 -> 5.08 mm
- net Net-(J1-Pad4): track 4.02 -> 8.73 mm
- net Net-(P2-Pad1): track 5.08 -> 9.72 mm
- net Net-(J1-Pad6): track 28.5 -> 25.2 mm
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Other:
- net class Default: trace_width 0.75 -> 0.4

Commit message: Schematics updates
Parts:
- removed P3: CONN_01X01, Pin_Headers:Pin_Header_Straight_1x01
Connections:
- U2 pad 33: Net-(U2-Pad33) -> Net-(J1-Pad4)
Routing:
- net Net-(J1-Pad4): track 8.73 -> 27.5 mm
Changed lines of the file:
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@@
     (links 28)
     (no_connects 0)
-    (area 0 0 0 0)
+    (area 143.481667 78.718999 181.54 133.195)
     (thickness 1.6)
     (drawings 0)
-    (tracks 86)
+    (tracks 94)
     (zones 0)
-    (modules 8)
-    (nets 40)
+    (modules 7)
+    (nets 39)
   )
   (page A4)
@@
     (visible_elements FFFFFF7F)
     (pcbplotparams
-      (layerselection 0x00030_80000001)
+      (layerselection 0x00000_00000001)
       (usegerberextensions false)
       (excludeedgelayer true)
@@
   (net 34 "Net-(U2-Pad22)")
   (net 35 "Net-(U2-Pad23)")
-  (net 36 "Net-(U2-Pad33)")
-  (net 37 "Net-(U2-Pad12)")
-  (net 38 "Net-(U2-Pad13)")
-  (net 39 "Net-(U2-Pad14)")
+  (net 36 "Net-(U2-Pad12)")
+  (net 37 "Net-(U2-Pad13)")
+  (net 38 "Net-(U2-Pad14)")
   (net_class Default "This is the default net class."
     (clearance 0.2)
@@
     (add_net "Net-(U2-Pad22)")
     (add_net "Net-(U2-Pad23)")
-    (add_net "Net-(U2-Pad33)")
     (add_net "Net-(U2-Pad9)")
   )
@@
       (net 3 "Net-(J1-Pad6)"))
     (pad 33 thru_hole circle (at -7.62 -2.54) (size 2 2) (drill 0.762) (layers *.Cu *.Mask F.SilkS)
-      (net 36 "Net-(U2-Pad33)"))
+      (net 1 "Net-(J1-Pad4)"))
     (pad 34 thru_hole circle (at -7.62 -5.08) (size 2 2) (drill 0.762) (layers *.Cu *.Mask F.SilkS)
       (net 2 "Net-(J1-Pad2)"))
@@
       (net 20 "Net-(U1-Pad1)"))
     (pad 12 thru_hole circle (at 7.62 5.08) (size 2 2) (drill 0.762) (layers *.Cu *.Mask F.SilkS)
-      (net 37 "Net-(U2-Pad12)"))
+      (net 36 "Net-(U2-Pad12)"))
     (pad 13 thru_hole circle (at 7.62 7.62) (size 2 2) (drill 0.762) (layers *.Cu *.Mask F.SilkS)
-      (net 38 "Net-(U2-Pad13)"))
+      (net 37 "Net-(U2-Pad13)"))
     (pad 14 thru_hole circle (at 7.62 10.16) (size 2 2) (drill 0.762) (layers *.Cu *.Mask F.SilkS)
-      (net 39 "Net-(U2-Pad14)"))
+      (net 38 "Net-(U2-Pad14)"))
   )
   (module Pin_Headers:Pin_Header_Straight_1x05 (layer F.Cu)
@@
     (model Pin_Headers.3dshapes/Pin_Header_Straight_1x05.wrl
       (at (xyz 0 -0.2 0))
-      (scale (xyz 1 1 1))
-      (rotate (xyz 0 0 90))
-    )
-  )
-  (module Pin_Headers:Pin_Header_Straight_1x01 (layer F.Cu)
-    (at 154.305 95.885)
-    (descr "Through hole pin header")
-    (tags "pin header")
-    (fp_text reference P3 (at 0 -5.1) (layer F.SilkS)
-      (effects (font (size 1 1) (thickness 0.15)))
-    )
-    (fp_text value CONN_01X01 (at 0 -3.1) (layer F.Fab)
-      (effects (font (size 1 1) (thickness 0.15)))
-    )
-    (fp_line (start 1.55 -1.55) (end 1.55 0) (layer F.SilkS) (width 0.15))
-    (fp_line (start -1.75 -1.75) (end -1.75 1.75) (layer F.CrtYd) (width 0.05))
-    (fp_line (start 1.75 -1.75) (end 1.75 1.75) (layer F.CrtYd) (width 0.05))
-    (fp_line (start -1.75 -1.75) (end 1.75 -1.75) (layer F.CrtYd) (width 0.05))
-    (fp_line (start -1.75 1.75) (end 1.75 1.75) (layer F.CrtYd) (width 0.05))
-    (fp_line (start -1.55 0) (end -1.55 -1.55) (layer F.SilkS) (width 0.15))
-    (fp_line (start -1.55 -1.55) (end 1.55 -1.55) (layer F.SilkS) (width 0.15))
-    (fp_line (start -1.27 1.27) (end 1.27 1.27) (layer F.SilkS) (width 0.15))
-    (pad 1 thru_hole rect (at 0 0) (size 2.2352 2.2352) (drill 1.016) (layers *.Cu *.Mask F.SilkS)
-      (net 1 "Net-(J1-Pad4)"))
-    (model Pin_Headers.3dshapes/Pin_Header_Straight_1x01.wrl
-      (at (xyz 0 0 0))
       (scale (xyz 1 1 1))
       (rotate (xyz 0 0 90))
@@
       (net 8 "Net-(J1-Pad7)"))
   )
-  (segment (start 153.162 87.63) (end 153.162 92.583) (width 0.4) (layer F.Cu) (net 1))
-  (segment (start 154.305 93.726) (end 154.305 95.885) (width 0.4) (layer F.Cu) (net 1))
-  (segment (start 153.162 92.583) (end 154.305 93.726) (width 0.4) (layer F.Cu) (net 1))
+  (segment (start 161.925 91.44) (end 161.925 91.821) (width 0.4) (layer F.Cu) (net 1))
+  (segment (start 156.845 86.36) (end 161.925 91.44) (width 0.4) (layer F.Cu) (net 1))
+  (segment (start 156.845 85.725) (end 156.845 86.36) (width 0.4) (layer F.Cu) (net 1))
+  (segment (start 156.21 85.09) (end 156.845 85.725) (width 0.4) (layer F.Cu) (net 1))
+  (segment (start 155.575 85.09) (end 156.21 85.09) (width 0.4) (layer F.Cu) (net 1))
+  (segment (start 153.162 87.503) (end 155.575 85.09) (width 0.4) (layer F.Cu) (net 1))
+  (segment (start 164.084 104.14) (end 165.1 104.14) (width 0.4) (layer F.Cu) (net 1))
+  (segment (start 162.052 102.108) (end 164.084 104.14) (width 0.4) (layer F.Cu) (net 1))
+  (segment (start 162.052 91.948) (end 162.052 102.108) (width 0.4) (layer F.Cu) (net 1))
+  (segment (start 161.925 91.821) (end 162.052 91.948) (width 0.4) (layer F.Cu) (net 1))
+  (segment (start 153.162 87.63) (end 153.162 87.503) (width 0.4) (layer F.Cu) (net 1))
   (segment (start 165.1 101.6) (end 163.83 101.6) (width 0.4) (layer F.Cu) (net 2))
   (segment (start 151.892 86.36) (end 150.622 87.63) (width 0.4) (layer F.Cu) (net 2))
@@
   (segment (start 156.21 82.55) (end 152.4 86.36) (width 0.4) (layer F.Cu) (net 2))
   (segment (start 161.29 82.55) (end 156.21 82.55) (width 0.4) (layer F.Cu) (net 2))
-  (segment (start 162.56 83.82) (end 161.29 82.55) (width 0.4) (layer F.Cu) (net 2))
-  (segment (start 162.56 100.33) (end 162.56 83.82) (width 0.4) (layer F.Cu) (net 2))
-  (segment (start 163.83 101.6) (end 162.56 100.33) (width 0.4) (layer F.Cu) (net 2))
+  (segment (start 163.195 83.82) (end 161.29 82.55) (width 0.4) (layer F.Cu) (net 2))
+  (segment (start 163.195 100.33) (end 163.195 83.82) (width 0.4) (layer F.Cu) (net 2))
+  (segment (start 163.83 101.6) (end 163.195 100.33) (width 0.4) (layer F.Cu) (net 2))
   (segment (start 155.702 87.63) (end 155.702 88.392) (width 0.4) (layer F.Cu) (net 3))
   (segment (start 155.702 88.392) (end 161.29 93.98) (width 0.4) (layer F.Cu) (net 3))
@@
   (segment (start 152.4 102.87) (end 151.13 101.6) (width 0.4) (layer F.Cu) (net 16))
   (segment (start 152.4 107.95) (end 152.4 102.87) (width 0.4) (layer F.Cu) (net 16))
-  (segment (start 172.72 85.09) (end 172.72 87.63) (width 0.4) (layer F.Cu) (net 17) (status 400000))
-  (segment (start 172.72 87.63) (end 175.26 90.17) (width 0.4) (layer F.Cu) (net 17) (status 800000))
+  (segment (start 172.72 85.09) (end 172.72 87.63) (width 0.4) (layer F.Cu) (net 17))
+  (segment (start 172.72 87.63) (end 175.26 90.17) (width 0.4) (layer F.Cu) (net 17))
   (segment (start 165.1 111.76) (end 166.37 111.76) (width 0.4) (layer F.Cu) (net 18))
   (segment (start 170.18 107.95) (end 170.18 85.09) (width 0.4) (layer F.Cu) (net 18) (status 20))
