File: BUG/WheelsAndIRT/WheelsAndIRT.sch (KiCad schematic (older format))
At the start: 8 parts, among them J1 RJ12, P1 CONN_01X05, P2 CONN_01X05, P3 CONN_01X01, P4 IRT, U1 uln2803A, U2 Arduino_Mini

Commit message: Update WheelsAndIRT
Parts:
- J1: footprint Connect:RJ12_E -> bugs:RJ12_Client
Connections:
- net at U1.7 (С7): now also U2.18 (10); no longer U2.30 (3)
- net at P4.2 (P2): now also U2.30 (3); no longer U2.18 (10)
- net at U2.34 (RXI): now also J1.2; no longer J1.1
- net at U2.35 (TXO): now also J1.1; no longer J1.2
Changed lines of the file:
@@
 LIBS:contrib
 LIBS:valves
-LIBS:bug-cache
+LIBS:WheelsAndIRT-cache
 EELAYER 25 0
 EELAYER END
@@
 F 0 "J1" H 6650 2350 50  0000 C CNN
 F 1 "RJ12" H 6300 2350 50  0000 C CNN
-F 2 "Connect:RJ12_E" H 6450 1850 50  0001 C CNN
+F 2 "bugs:RJ12_Client" H 6450 1850 50  0001 C CNN
 F 3 "" H 6450 1850 50  0000 C CNN
 	1    6450 1850
@@
 	4300 3650 4150 3650
 Wire Wire Line
-	4150 3550 4300 3550
-Wire Wire Line
 	4300 3450 4150 3450
 Connection ~ 3200 3350
@@
 Wire Wire Line
 	4250 3150 4300 3150
-Wire Wire Line
-	4300 1750 4300 3050
 Connection ~ 3200 3200
 Wire Wire Line
@@
 	2800 3200 3200 3200
 Wire Wire Line
-	6000 1750 4300 1750
-Wire Wire Line
-	4250 3150 4250 1650
-Wire Wire Line
-	4250 1650 6000 1650
+	4250 1750 6000 1750
 Wire Wire Line
 	4200 2150 6000 2150
@@
 	5900 3250 5800 3250
 Wire Wire Line
-	5800 3250 5800 4150
-Wire Wire Line
-	5800 4150 5400 4150
+	5800 3250 5800 4650
+Wire Wire Line
+	4250 1750 4250 3150
+Wire Wire Line
+	4300 3050 4300 1650
+Wire Wire Line
+	4300 1650 6000 1650
+Wire Wire Line
+	5400 4150 5450 4150
+Wire Wire Line
+	5450 4150 5450 4750
+Wire Wire Line
+	5450 4750 4200 4750
+Wire Wire Line
+	4200 4750 4200 3550
+Wire Wire Line
+	4200 3550 4150 3550
+Wire Wire Line
+	4300 3550 4300 4650
+Wire Wire Line
+	4300 4650 5800 4650
 $EndSCHEMATC

Commit message: Schematics updates
Parts:
- removed P3: CONN_01X01, Pin_Headers:Pin_Header_Straight_1x01, symbol CONN_01X01
Connections:
- net at U2.33 (RST): now also J1.4
Changed lines of the file:
@@
 Text Label 6200 2150 0    60   ~ 0
 GND
-$Comp
-L CONN_01X01 P3
-U 1 1 57485E22
-P 5750 1950
-F 0 "P3" H 5750 2050 50  0000 C CNN
-F 1 "CONN_01X01" V 5850 1950 50  0000 C CNN
-F 2 "Pin_Headers:Pin_Header_Straight_1x01" H 5750 1950 50  0001 C CNN
-F 3 "" H 5750 1950 50  0000 C CNN
-	1    5750 1950
-	-1   0    0    1
-$EndComp
 Wire Wire Line
 	4300 3850 4150 3850
@@
 Connection ~ 4200 3350
 Wire Wire Line
-	5950 1950 6000 1950
+	4050 1950 6000 1950
 $Comp
 L Arduino_Mini U2
@@
 Wire Wire Line
 	4300 4650 5800 4650
+Wire Wire Line
+	4300 3250 4050 3250
+Wire Wire Line
+	4050 3250 4050 1950
 $EndSCHEMATC
