File: matherboard/matherboard.sch (KiCad schematic (older format))
At the start: 17 parts, among them J1 RJ12, J2 RJ12, J3 RJ12, P1 VCC/GND, P2 CONN_01X02, P3 CONN_01X02, P4 CONN_01X02, P5 CONN_01X05, P6 CONN_01X02, U3 STAB3.3, U4 ESP8266

Commit message: Components for BUG
Parts:
- removed P1: VCC/GND, Pin_Headers:Pin_Header_Straight_1x02, symbol CONN_01X02
- added CON1: BARREL_JACK, Connect:BARREL_JACK, symbol BARREL_JACK
- added U1: button, bugs:button, symbol button
Connections:
- wire segments 72 -> 78
Changed lines of the file:
@@
-$EndComp
-$Comp
-L CONN_01X02 P1
-U 1 1 5739B957
-P 1500 1300
-F 0 "P1" H 1500 1450 50  0000 C CNN
-F 1 "VCC/GND" V 1600 1300 50  0000 C CNN
-F 2 "Pin_Headers:Pin_Header_Straight_1x02" H 1500 1300 50  0001 C CNN
-F 3 "" H 1500 1300 50  0000 C CNN
-	1    1500 1300
-	-1   0    0    1
 $EndComp
 $Comp
@@
 	2950 1350 3450 1350
 Wire Wire Line
-	3050 1350 3050 1050
-Wire Wire Line
-	3050 1050 1700 1050
-Wire Wire Line
-	1700 1050 1700 1250
+	3050 1050 3050 1350
+Wire Wire Line
+	1050 1050 3050 1050
 Wire Wire Line
 	2500 1700 2950 1700
@@
 	3050 1800 3050 1550
 Wire Notes Line
-	3200 850  3200 1950
-Wire Notes Line
-	1300 850  1300 1950
-Wire Notes Line
 	5600 1250 5600 4350
 Wire Notes Line
@@
 	1850 1350 2050 1350
 Wire Wire Line
-	1700 1350 1750 1350
-Wire Notes Line
-	1300 850  3200 850
-Wire Notes Line
-	1300 1950 3200 1950
+	1500 1350 1750 1350
+Wire Notes Line
+	850  850  3200 850
 Wire Wire Line
 	3650 1400 3650 3450
@@
 Connection ~ 3650 3400
 Connection ~ 3700 3350
+$Comp
+L button U1
+U 1 1 57487031
+P 1400 1650
+F 0 "U1" V 1600 1600 60  0000 C CNN
+F 1 "button" V 1200 1550 60  0000 C CNN
+F 2 "bugs:button" H 1450 1650 60  0001 C CNN
+F 3 "" H 1450 1650 60  0000 C CNN
+	1    1400 1650
+	1    0    0    -1
+$EndComp
+Wire Wire Line
+	1200 1250 1400 1250
+Wire Wire Line
+	1400 1250 1400 1350
+Wire Notes Line
+	850  850  850  2150
+Wire Notes Line
+	850  2150 1650 2150
+Wire Notes Line
+	1650 2150 1650 1850
+Wire Notes Line
+	1650 1850 3200 1850
+Wire Notes Line
+	3200 1850 3200 850
+$Comp
+L BARREL_JACK CON1
+U 1 1 57487687
+P 450 1200
+F 0 "CON1" H 450 1450 50  0000 C CNN
+F 1 "BARREL_JACK" H 450 1000 50  0000 C CNN
+F 2 "Connect:BARREL_JACK" H 450 1200 50  0001 C CNN
+F 3 "" H 450 1200 50  0000 C CNN
+	1    450  1200
+	1    0    0    -1
+$EndComp
+Wire Wire Line
+	750  1100 1200 1100
+Wire Wire Line
+	1200 1100 1200 1250
+Wire Wire Line
+	750  1300 1050 1300
+Wire Wire Line
+	1050 1300 1050 1050
+Wire Wire Line
+	750  1200 1050 1200
+Connection ~ 1050 1200
 $EndSCHEMATC

Commit message: Added power led to marherboard
Parts:
- added D1: LED, LEDs:LED-3MM, symbol LED
- added R5: 500, w_pth_resistors:rc03_vert, symbol R
Connections:
- wire segments 78 -> 82
Changed lines of the file:
@@
 	3700 1450 6100 1450
-Wire Wire Line
-	2050 1350 2050 1800
 Wire Wire Line
 	2950 1350 3450 1350
@@
 Connection ~ 3050 1350
 Wire Wire Line
-	2050 1800 3050 1800
+	2000 1800 3050 1800
 Wire Wire Line
 	3050 1800 3050 1550
@@
 	750  1200 1050 1200
 Connection ~ 1050 1200
+Wire Wire Line
+	2000 1000 2000 1800
+Connection ~ 2000 1350
+$Comp
+L LED D1
+U 1 1 574DB2B9
+P 1650 800
+F 0 "D1" H 1650 900 50  0000 C CNN
+F 1 "LED" H 1650 700 50  0000 C CNN
+F 2 "LEDs:LED-3MM" H 1650 800 50  0001 C CNN
+F 3 "" H 1650 800 50  0000 C CNN
+	1    1650 800
+	0    1    1    0
+$EndComp
+Wire Wire Line
+	2000 1000 1650 1000
+Wire Wire Line
+	1650 600  2150 600
+Wire Wire Line
+	2150 600  2150 700
+Wire Wire Line
+	2150 1000 2150 1050
+Connection ~ 2150 1050
+$Comp
+L R R5
+U 1 1 574DB6C9
+P 2150 850
+F 0 "R5" V 2230 850 50  0000 C CNN
+F 1 "500" V 2150 850 50  0000 C CNN
+F 2 "w_pth_resistors:rc03_vert" V 2080 850 50  0001 C CNN
+F 3 "" H 2150 850 50  0000 C CNN
+	1    2150 850
+	1    0    0    -1
+$EndComp
 $EndSCHEMATC

Commit message: Schematics updates
Parts:
- removed P5: CONN_01X05, Pin_Headers:Pin_Header_Straight_1x05, symbol CONN_01X05
- added P5: CONN_01X04, Pin_Headers:Pin_Header_Straight_1x04, symbol CONN_01X04
Connections:
- wire segments 82 -> 87
Changed lines of the file:
@@
 DTR
-$Comp
-L CONN_01X05 P5
-U 1 1 573B5742
-P 4200 1650
-F 0 "P5" H 4200 1950 50  0000 C CNN
-F 1 "CONN_01X05" V 4300 1650 50  0000 C CNN
-F 2 "Pin_Headers:Pin_Header_Straight_1x05" H 4200 1650 50  0001 C CNN
-F 3 "" H 4200 1650 50  0000 C CNN
-	1    4200 1650
-	0    -1   -1   0
-$EndComp
 $Comp
 L CONN_01X02 P3
@@
 Connection ~ 3650 2000
 Wire Wire Line
-	4100 1950 4100 1850
-Wire Wire Line
-	3050 1950 4100 1950
+	4100 1800 4100 1950
+Wire Wire Line
+	4100 1950 3050 1950
 Wire Wire Line
 	3650 2350 3800 2350
@@
 Wire Wire Line
 	6100 1450 6100 2550
+$Comp
+L CONN_01X04 P5
+U 1 1 5750347D
+P 4400 750
+F 0 "P5" H 4400 1000 50  0000 C CNN
+F 1 "CONN_01X04" V 4500 750 50  0000 C CNN
+F 2 "Pin_Headers:Pin_Header_Straight_1x04" H 4400 750 50  0001 C CNN
+F 3 "" H 4400 750 50  0000 C CNN
+	1    4400 750
+	0    -1   -1   0
+$EndComp
+Wire Wire Line
+	4250 950  4250 1400
+Connection ~ 4250 1400
+Wire Wire Line
+	4350 950  4350 1150
+Connection ~ 4350 1150
+Wire Wire Line
+	4450 950  4450 1450
+Connection ~ 4450 1450
+Wire Wire Line
+	4100 1800 4550 1800
+Wire Wire Line
+	4550 1800 4550 950
 $EndSCHEMATC
