File: BUG/DCDriver/DCDriver.sch (KiCad schematic (older format))
At the start: 8 parts, among them J1 RJ12, P1 W2, P2 W1, U1 L293D, U2 Arduino_Mini

Commit message: Many uodates
Parts:
- added P3: CONN_01X03, Pin_Headers:Pin_Header_Straight_1x03, symbol CONN_01X03
- added R4: R, Resistors_SMD:R_1206, symbol R
Connections:
- net at U2.18 (10): now also P3.3 (P3); no longer J1.4
- net at U2.9 (RST): now also R4.1
- new net: J1.4, P3.2 (P2)
- new net: P3.1 (P1), R4.2
Changed lines of the file:
@@
 	5550 4700 5800 4700
 Wire Wire Line
-	5750 3450 5750 4700
+	5750 3400 5750 4700
 Wire Wire Line
 	4500 3650 4500 4050
@@
 Wire Wire Line
 	9000 3900 8150 3900
-Wire Wire Line
-	9000 4850 9000 3900
-Wire Wire Line
-	6300 4850 9000 4850
-Wire Wire Line
-	6300 2400 6300 4850
 Wire Wire Line
 	8300 3700 8150 3700
@@
 Connection ~ 6350 3100
 Wire Wire Line
-	6550 2450 6550 3100
-Wire Wire Line
-	8350 2450 6550 2450
+	6550 3100 6550 2450
+Wire Wire Line
+	6550 2450 8350 2450
 Wire Wire Line
 	8150 3100 8350 3100
 Wire Wire Line
-	6550 3100 5750 3100
+	5750 3100 6550 3100
 Wire Wire Line
 	6350 4400 6350 3100
@@
 	4750 3400 4750 3500
 Wire Wire Line
-	5750 3400 5750 3500
+	5750 3450 5750 3500
 Wire Wire Line
 	6000 3300 5750 3300
@@
 $EndComp
 Wire Wire Line
-	8350 2550 8350 2450
+	8350 2450 8350 2550
 Wire Wire Line
 	8350 3100 8350 2850
+$Comp
+L CONN_01X03 P3
+U 1 1 5788E7BD
+P 7050 1950
+F 0 "P3" H 7050 2150 50  0000 C CNN
+F 1 "CONN_01X03" V 7150 1950 50  0000 C CNN
+F 2 "Pin_Headers:Pin_Header_Straight_1x03" H 7050 1950 50  0001 C CNN
+F 3 "" H 7050 1950 50  0000 C CNN
+	1    7050 1950
+	0    -1   -1   0
+$EndComp
+Wire Wire Line
+	6300 2400 6300 2700
+Wire Wire Line
+	6300 2700 7050 2700
+Wire Wire Line
+	7050 2700 7050 2150
+Wire Wire Line
+	9000 3900 9000 2150
+Wire Wire Line
+	9000 2150 7150 2150
+Wire Wire Line
+	6950 2150 6800 2150
+Wire Wire Line
+	6800 2150 6800 1750
+Wire Wire Line
+	6800 1750 8650 1750
+Wire Wire Line
+	8650 3000 8150 3000
+$Comp
+L R R4
+U 1 1 5788EB3C
+P 8650 2600
+F 0 "R4" V 8730 2600 50  0000 C CNN
+F 1 "R" V 8650 2600 50  0000 C CNN
+F 2 "Resistors_SMD:R_1206" V 8580 2600 50  0001 C CNN
+F 3 "" H 8650 2600 50  0000 C CNN
+	1    8650 2600
+	-1   0    0    1
+$EndComp
+Wire Wire Line
+	8650 2750 8650 3000
+Wire Wire Line
+	8650 1750 8650 2450
 $EndSCHEMATC
