File: BUG/Driver/Driver.sch (KiCad schematic (older format))
At the start: 6 parts, among them J1 RJ12, P1 CONN_01X05, P2 CONN_01X05, P3 CONN_01X03, U1 uln2803A, U2 Arduino_Mini

Commit message: Many uodates
Parts:
- added R1: 0, Resistors_SMD:R_1206, symbol R
Connections:
- net at P1.5 (P5), P2.5 (P5), U1.10 (COM): now also R1.2
- net at J1.1, U2.7 (RAW): now also R1.1
Changed lines of the file:
@@
 	4750 3650 4550 3650
-Wire Wire Line
-	3550 3450 3550 3550
 Wire Wire Line
 	3500 3550 3650 3550
@@
 	5100 2000 5100 2400
 Wire Wire Line
-	5100 2400 5900 2400
+	3550 2400 5900 2400
 Wire Wire Line
 	5900 2400 5900 3250
@@
 Wire Wire Line
 	6700 3450 5850 3450
+Connection ~ 3550 3450
+Connection ~ 5100 2400
+$Comp
+L R R1
+U 1 1 57878168
+P 3550 2800
+F 0 "R1" V 3630 2800 50  0000 C CNN
+F 1 "0" V 3550 2800 50  0000 C CNN
+F 2 "Resistors_SMD:R_1206" V 3480 2800 50  0001 C CNN
+F 3 "" H 3550 2800 50  0000 C CNN
+	1    3550 2800
+	1    0    0    -1
+$EndComp
+Wire Wire Line
+	3550 2950 3550 3550
+Wire Wire Line
+	3550 2650 3550 2400
 $EndSCHEMATC
