File: BUG/Matherboard2/matherboard2.kicad_pcb (KiCad board)
At the start: 2 copper layers, 38 parts, among them CON1 BARREL_JACK, J1 RJ12, J2 RJ12, J3 RJ12, P1 ON/OFF, P2 FW, P3 RXTX, U1 BUTTON, U2 AP1117-5, U3 ESP-201, U4 AP1117-3

Commit message: Many uodates
Parts:
- removed J3: RJ12, Connect:RJ12_E
- added P4: GND, Pin_Headers:Pin_Header_Straight_1x01, F.Cu at (157.5, 149.6)
- added R27: 0, Resistors_SMD:R_1206, F.Cu at (183.5, 104.1)
- added R28: 0, Resistors_SMD:R_1206, F.Cu at (188.0, 104.1)
- added R29: 0, Resistors_SMD:R_1206, F.Cu at (192.4, 104.1)
- added R30: 0, Resistors_SMD:R_1206, F.Cu at (170.4, 101.1)
- added R31: 0, Resistors_SMD:R_1206, F.Cu at (183.5, 101.0)
- added R32: 0, Resistors_SMD:R_1206, F.Cu at (188.0, 101.0)
- added R33: 0, Resistors_SMD:R_1206, F.Cu at (183.5, 97.8)
- added R34: 0, Resistors_SMD:R_1206, F.Cu at (170.4, 105.2)
- J1, J2: value RJ12 -> RJ12double; footprint Connect:RJ12_E -> bugs:RJ12double
- U2, U4: footprint Buttons_Switches_ThroughHole:SW_Micro_SPST -> bugs:SMD-stab
- moved R5 38.4 mm to (183.4, 136.1)
- moved R10 38.4 mm to (192.8, 142.7)
- moved R12 38.4 mm to (188.0, 139.4)
- moved R9 38.4 mm to (188.2, 142.7)
- moved R11 38.4 mm to (183.6, 139.4)
- moved R8 38.4 mm to (183.6, 142.7)
- moved R23 37.9 mm to (170.2, 138.9)
- moved J1 37.4 mm to (186.7, 138.4)
- moved J2 26.2 mm to (186.7, 111.8)
- moved R14 10.8 mm to (188.0, 130.4)
- moved R15 10.8 mm to (192.8, 130.4)
- moved R13 10.8 mm to (183.6, 130.4)
- moved R17 10.8 mm to (188.0, 127.1)
- moved R16 10.8 mm to (183.6, 127.1)
- moved R6 10.6 mm to (183.6, 124.2)
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Connections:
- P1 pad 2: Net-(J1-Pad1) -> Net-(P1-Pad2)
- R11 pad 1: Net-(J1-Pad5) -> Net-(J1-Pad13)
- R13 pad 1: Net-(J2-Pad3) -> Net-(J1-Pad3)
- R16 pad 1: Net-(J2-Pad5) -> Net-(J1-Pad5)
- R18 pad 1: Net-(J3-Pad3) -> Net-(J2-Pad11)
- R21 pad 1: Net-(J3-Pad5) -> Net-(J2-Pad13)
- R23 pad 1: Net-(J1-Pad4) -> Net-(J1-Pad12)
- R24 pad 1: Net-(J2-Pad4) -> Net-(J1-Pad4)
- R25 pad 1: Net-(J3-Pad4) -> Net-(J2-Pad12)
- R5 pad 1: Net-(J1-Pad6) -> Net-(J1-Pad14)
- R6 pad 1: Net-(J2-Pad6) -> Net-(J1-Pad6)
- R7 pad 1: Net-(J3-Pad6) -> Net-(J2-Pad14)
- R8 pad 1: Net-(J1-Pad3) -> Net-(J1-Pad11)
- U2 pad 3: Net-(J1-Pad1) -> Net-(P1-Pad2)
- U3 pad 12: Net-(R23-Pad2) -> Net-(R25-Pad2)
- U3 pad 13: Net-(R25-Pad2) -> Net-(R24-Pad2)
- U3 pad 18: Net-(R24-Pad2) -> Net-(R23-Pad2)
Routing:
- net Net-(R30-Pad2): track 0.00 -> 171.9 mm
- net Net-(P1-Pad2): track 0.00 -> 38.1 mm
- net Net-(R23-Pad2): track 66.1 -> 92.3 mm
- net Net-(J1-Pad1): track 105.7 -> 80.3 mm
- net Net-(CON1-Pad2): track 151.5 -> 167.7 mm
- net Net-(R24-Pad2): track 88.4 -> 74.4 mm
- net Net-(R12-Pad2): track 109.6 -> 120.2 mm
- net Net-(R26-Pad2): track 2.36 -> 12.2 mm
- net Net-(R33-Pad2): track 106.4 -> 115.8 mm
- net Net-(J2-Pad14): track 0.00 -> 8.95 mm
- net Net-(J1-Pad14): track 0.00 -> 8.19 mm
- net Net-(R10-Pad2): track 96.7 -> 104.1 mm
- net Net-(J1-Pad11): track 0.00 -> 6.89 mm
- net Net-(R3-Pad1): track 46.6 -> 39.8 mm
- net Net-(J1-Pad13): track 0.00 -> 6.36 mm
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