File: kidkit/kidkit.sch (KiCad schematic (older format))
At the start: 15 parts, among them P4 CONN_01X02, P7 CONN_01X02, U2 Arduino_Mini, U3 SPX2920U-3.3, U4 ESP8266

Commit message: Modified kidkit scheme
Parts:
- added P?: CONN_01X04, symbol CONN_01X04
- added P?: CONN_01X08, symbol CONN_01X08
- added P? (x5): CONN_01X02, symbol CONN_01X02
- added P?: CONN_01X03, symbol CONN_01X03
Connections:
- wire segments 102 -> 152
Changed lines of the file:
@@
+$EndComp
+$Comp
+L L293D U?
+U 1 1 587DD6FF
+P 2600 3650
+F 0 "U?" H 2900 4150 60  0000 C CNN
+F 1 "L293D" H 2600 4150 60  0000 C CNN
+F 2 "" H 3150 3300 60  0000 C CNN
+F 3 "" H 3150 3300 60  0000 C CNN
+	1    2600 3650
+	1    0    0    -1
+$EndComp
+$Comp
+L CONN_01X02 P?
+U 1 1 587DE3C0
+P 1500 3550
+F 0 "P?" H 1500 3700 50  0000 C CNN
+F 1 "CONN_01X02" V 1600 3550 50  0000 C CNN
+F 2 "" H 1500 3550 50  0000 C CNN
+F 3 "" H 1500 3550 50  0000 C CNN
+	1    1500 3550
+	-1   0    0    1
+$EndComp
+$Comp
+L CONN_01X02 P?
+U 1 1 587DE533
+P 1500 4000
+F 0 "P?" H 1500 4150 50  0000 C CNN
+F 1 "CONN_01X02" V 1600 4000 50  0000 C CNN
+F 2 "" H 1500 4000 50  0000 C CNN
+F 3 "" H 1500 4000 50  0000 C CNN
+	1    1500 4000
+	-1   0    0    1
+$EndComp
+$Comp
+L CONN_01X04 P?
+U 1 1 587DEA8E
+P 1900 1700
+F 0 "P?" H 1900 1950 50  0000 C CNN
+F 1 "CONN_01X04" V 2000 1700 50  0000 C CNN
+F 2 "" H 1900 1700 50  0000 C CNN
+F 3 "" H 1900 1700 50  0000 C CNN
+	1    1900 1700
+	-1   0    0    1
 $EndComp
 $Comp
@@
 $EndComp
 $Comp
-L L293D U?
-U 1 1 587DD6FF
-P 2600 3650
-F 0 "U?" H 2900 4150 60  0000 C CNN
-F 1 "L293D" H 2600 4150 60  0000 C CNN
-F 2 "" H 3150 3300 60  0000 C CNN
-F 3 "" H 3150 3300 60  0000 C CNN
-	1    2600 3650
-	1    0    0    -1
+L CONN_01X08 P?
+U 1 1 587E510C
+P 4900 5500
+F 0 "P?" H 4900 5950 50  0000 C CNN
+F 1 "CONN_01X08" V 5000 5500 50  0000 C CNN
+F 2 "" H 4900 5500 50  0000 C CNN
+F 3 "" H 4900 5500 50  0000 C CNN
+	1    4900 5500
+	0    1    1    0
+$EndComp
+$Comp
+L CONN_01X02 P?
+U 1 1 587E5CCD
+P 4450 6500
+F 0 "P?" H 4450 6650 50  0000 C CNN
+F 1 "CONN_01X02" V 4550 6500 50  0000 C CNN
+F 2 "" H 4450 6500 50  0000 C CNN
+F 3 "" H 4450 6500 50  0000 C CNN
+	1    4450 6500
+	0    1    1    0
+$EndComp
+$Comp
+L CONN_01X02 P?
+U 1 1 587E5DE2
+P 4900 6250
+F 0 "P?" H 4900 6400 50  0000 C CNN
+F 1 "CONN_01X02" V 5000 6250 50  0000 C CNN
+F 2 "" H 4900 6250 50  0000 C CNN
+F 3 "" H 4900 6250 50  0000 C CNN
+	1    4900 6250
+	0    1    1    0
+$EndComp
+$Comp
+L CONN_01X02 P?
+U 1 1 587E5E3D
+P 4150 6500
+F 0 "P?" H 4150 6650 50  0000 C CNN
+F 1 "CONN_01X02" V 4250 6500 50  0000 C CNN
+F 2 "" H 4150 6500 50  0000 C CNN
+F 3 "" H 4150 6500 50  0000 C CNN
+	1    4150 6500
+	0    1    1    0
+$EndComp
+$Comp
+L CONN_01X02 P?
+U 1 1 587E5F52
+P 5900 6250
+F 0 "P?" H 5900 6400 50  0000 C CNN
+F 1 "CONN_01X02" V 6000 6250 50  0000 C CNN
+F 2 "" H 5900 6250 50  0000 C CNN
+F 3 "" H 5900 6250 50  0000 C CNN
+	1    5900 6250
+	0    1    1    0
+$EndComp
+$Comp
+L CONN_01X02 P?
+U 1 1 587E5FE3
+P 5550 6250
+F 0 "P?" H 5550 6400 50  0000 C CNN
+F 1 "CONN_01X02" V 5650 6250 50  0000 C CNN
+F 2 "" H 5550 6250 50  0000 C CNN
+F 3 "" H 5550 6250 50  0000 C CNN
+	1    5550 6250
+	0    1    1    0
+$EndComp
+$Comp
+L CONN_01X03 P?
+U 1 1 587E620C
+P 6250 6000
+F 0 "P?" H 6250 6200 50  0000 C CNN
+F 1 "CONN_01X03" V 6350 6000 50  0000 C CNN
+F 2 "" H 6250 6000 50  0000 C CNN
+F 3 "" H 6250 6000 50  0000 C CNN
+	1    6250 6000
+	0    1    1    0
 $EndComp
 Wire Wire Line
@@
 	5400 2400 6300 2400
 Wire Wire Line
-	4300 4050 4150 4050
+	4100 4050 4300 4050
 Wire Wire Line
 	3900 3450 4300 3450
@@
 	5000 1050 5000 1300
 Wire Wire Line
-	5400 3350 5550 3350
+	5400 3350 6350 3350
 Wire Wire Line
 	5000 1400 5000 2000
 Wire Wire Line
-	3200 2000 5650 2000
-Wire Wire Line
 	5650 2000 5650 2400
-Connection ~ 5000 2000
 Wire Wire Line
 	6400 2550 5750 2550
@@
 	1900 2250 4150 2250
 Wire Wire Line
-	4150 2250 4150 3350
+	4150 1850 4150 3350
 Connection ~ 1900 3650
 Wire Wire Line
@@
 	5200 2600 5550 2600
 Wire Wire Line
-	5550 2600 5550 3350
+	5550 1550 5550 5300
 Connection ~ 3450 3300
-$Comp
-L CONN_01X02 P?
-U 1 1 587DE3C0
-P 1500 3550
-F 0 "P?" H 1500 3700 50  0000 C CNN
-F 1 "CONN_01X02" V 1600 3550 50  0000 C CNN
-F 2 "" H 1500 3550 50  0000 C CNN
-F 3 "" H 1500 3550 50  0000 C CNN
-	1    1500 3550
-	-1   0    0    1
-$EndComp
-$Comp
-L CONN_01X02 P?
-U 1 1 587DE533
-P 1500 4000
-F 0 "P?" H 1500 4150 50  0000 C CNN
-F 1 "CONN_01X02" V 1600 4000 50  0000 C CNN
-F 2 "" H 1500 4000 50  0000 C CNN
-F 3 "" H 1500 4000 50  0000 C CNN
-	1    1500 4000
-	-1   0    0    1
-$EndComp
 Wire Wire Line
 	2100 3500 1700 3500
@@
 Wire Wire Line
 	1800 3950 1700 3950
+Wire Wire Line
+	5000 2000 5650 2000
+Wire Wire Line
+	2100 1550 5550 1550
+Connection ~ 5550 2600
+Wire Wire Line
+	2100 1850 4150 1850
+Connection ~ 4150 2250
+Wire Wire Line
+	2100 1650 4100 1650
+Wire Wire Line
+	4100 1650 4100 4050
+Wire Wire Line
+	2100 1750 5500 1750
+Wire Wire Line
+	5500 1750 5500 3450
+Wire Wire Line
+	5500 3450 5400 3450
+Wire Wire Line
+	5550 5300 5250 5300
+Connection ~ 5550 3350
+Wire Wire Line
+	5150 5300 5150 5200
+Wire Wire Line
+	5150 5200 4150 5200
+Wire Wire Line
+	4150 5200 4150 4150
+Wire Wire Line
+	5050 5300 5050 5150
+Wire Wire Line
+	5050 5150 4250 5150
+Wire Wire Line
+	4250 3350 4250 6300
+Connection ~ 4250 3350
+Wire Wire Line
+	5400 3950 5600 3950
+Wire Wire Line
+	5600 3950 5600 5100
+Wire Wire Line
+	5600 5100 4850 5100
+Wire Wire Line
+	4850 5100 4850 5300
+Wire Wire Line
+	4750 5300 4750 5000
+Wire Wire Line
+	4750 5000 5500 5000
+Wire Wire Line
+	5500 5000 5500 4050
+Wire Wire Line
+	5500 4050 5400 4050
+Wire Wire Line
+	4650 5300 4650 5050
+Wire Wire Line
+	4650 5050 5650 5050
+Wire Wire Line
+	5650 5050 5650 3850
+Wire Wire Line
+	5650 3850 5400 3850
+Wire Wire Line
+	4550 5300 4550 4800
+Wire Wire Line
+	4550 4800 5400 4800
+Wire Wire Line
+	5400 4800 5400 4150
+Wire Wire Line
+	4700 4600 4500 4600
+Wire Wire Line
+	4500 4600 4500 6300
+Wire Wire Line
+	4200 6300 4400 6300
+Wire Wire Line
+	4100 6300 4100 6200
+Wire Wire Line
+	4100 6200 4500 6200
+Connection ~ 4500 6200
+Connection ~ 4250 6300
+Connection ~ 4250 5150
+Wire Wire Line
+	4950 6050 4950 4600
+Wire Wire Line
+	4950 4600 4800 4600
+Connection ~ 4850 6050
+Wire Wire Line
+	5500 6050 5500 5950
+Wire Wire Line
+	5500 5950 4250 5950
+Connection ~ 4250 5950
+Wire Wire Line
+	5850 6050 5850 5900
+Wire Wire Line
+	5850 5900 4250 5900
+Connection ~ 4250 5900
+Wire Wire Line
+	5600 6050 5600 5600
+Wire Wire Line
+	5600 5600 5800 5600
+Wire Wire Line
+	5800 5600 5800 3650
+Wire Wire Line
+	5800 3650 5400 3650
+Wire Wire Line
+	5950 6050 5950 3550
+Wire Wire Line
+	5950 3550 5400 3550
+Wire Wire Line
+	6150 5800 6150 3750
+Wire Wire Line
+	6150 3750 5400 3750
+Wire Wire Line
+	6350 3350 6350 5800
+Wire Wire Line
+	6250 5800 4250 5800
+Connection ~ 4250 5800
 $EndSCHEMATC
