File: EduKit/EduKit.kicad_pcb (KiCad board)
At the start: 2 copper layers, 25 parts, among them P1 Wheel, P10 BlueLED, P11 IRReceiver, P2 Wheel, P3 Sonar, P4 PowerPINs, P5 Headlight, P6 Headlight, P7 RCReader, P8 IRTransmitter, P9 RedLED, U1 L293D, U2 Arduino_Mini, U3 SPX2920U-3.3, U4 ESP8266, U5 PowerButton

Commit message: Jackalized a little
Parts:
- moved U1 6.47 mm to (125.2, 112.3), turned to 270 degrees
- moved P11 6.27 mm to (126.5, 60.7), turned to 270 degrees
- moved P8 4.02 mm to (162.1, 60.7), turned to 270 degrees
- moved P1 3.66 mm to (108.0, 94.9)
- moved P5 3.59 mm to (111.3, 64.5)
- moved P6 3.59 mm to (169.7, 62.0)
- moved P2 3.41 mm to (172.2, 92.5), turned to 0 degrees
- moved P3 2.34 mm to (144.3, 60.7)
- moved C1 1.14 mm to (162.1, 101.3)
- moved D2 1.14 mm to (172.2, 116.6)
- moved P9 1.14 mm to (127.8, 84.8)
- moved U3 1.14 mm to (159.5, 96.3)
- moved U4 1.14 mm to (162.1, 119.1)
- moved P10 1.14 mm to (124.0, 84.8)
- moved D1 1.14 mm to (172.2, 121.7)
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Routing:
- net Net-(P10-Pad2): track 1.27 -> 108.1 mm
- net Net-(P5-Pad2): track 0.00 -> 68.6 mm
- net Net-(P3-Pad2): track 0.00 -> 45.3 mm
- net Net-(D3-Pad2): track 20.3 -> 60.0 mm
- net Net-(P9-Pad1): track 0.00 -> 37.2 mm
- net Net-(P1-Pad1): track 0.00 -> 22.7 mm
- net Net-(P1-Pad2): track 0.00 -> 19.9 mm
- net Net-(P4-Pad1): track 0.00 -> 19.3 mm
- net Net-(C1-Pad2): track 134.2 -> 147.4 mm
- net Net-(U1-Pad2): track 0.00 -> 12.4 mm
- net Net-(P11-Pad1): track 0.00 -> 10.2 mm
- net Net-(D3-Pad1): track 0.00 -> 8.89 mm
- net Net-(U1-Pad1): track 0.00 -> 8.77 mm
Other:
- net class Default: trace_width 0.75 -> 0.4

Commit message: Some fixes
Parts:
- moved P7 4.10 mm to (152.4, 102.9)
Routing:
- net Net-(U1-Pad7): track 0.00 -> 55.2 mm
- net Net-(P10-Pad2): track 108.1 -> 146.2 mm
- net Net-(U1-Pad9): track 0.00 -> 35.3 mm
- net Net-(U1-Pad10): track 0.00 -> 33.2 mm
- net Net-(P7-Pad7): track 0.00 -> 27.6 mm
- net Net-(U1-Pad15): track 0.00 -> 21.0 mm
- net Net-(P7-Pad6): track 0.00 -> 7.06 mm
- net Net-(P7-Pad5): track 0.00 -> 7.06 mm
- net Net-(P7-Pad8): track 0.00 -> 6.01 mm

Commit message: Jackalized a little
Parts:
- P10: value BlueLED -> Speaker
- moved P1 71.2 mm to (179.1, 97.8), turned to 180 degrees
- moved P2 67.1 mm to (105.3, 96.9), turned to 180 degrees
- moved P9 46.9 mm to (166.1, 57.9), turned to 90 degrees
- moved P7 28.6 mm to (151.8, 131.4), turned to 270 degrees
- moved P10 26.3 mm to (144.1, 67.9)
- moved R5 24.7 mm to (167.6, 83.8), turned to 0 degrees
- moved U2 21.6 mm to (125.2, 84.8)
- moved C1 21.6 mm to (148.1, 84.8)
- moved D2 21.6 mm to (158.2, 100.1)
- moved R1 21.6 mm to (150.6, 107.7)
- moved U3 21.6 mm to (145.5, 79.8)
- moved U4 21.6 mm to (148.1, 102.6)
- moved D1 21.6 mm to (158.2, 105.2)
- moved R2 21.6 mm to (145.5, 92.5)
- moved R3 21.6 mm to (148.1, 92.5)
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Routing:
- net Net-(U1-Pad1): track 8.77 -> 76.2 mm
- net Net-(P5-Pad2): track 68.6 -> 134.8 mm
- net Net-(P10-Pad2): track 146.2 -> 81.7 mm
- net Net-(P2-Pad2): track 0.00 -> 60.8 mm
- net Net-(U1-Pad7): track 55.2 -> 0.18 mm
- net Net-(P2-Pad1): track 0.00 -> 53.2 mm
- net Net-(P1-Pad2): track 19.9 -> 72.7 mm
- net Net-(U1-Pad15): track 21.0 -> 73.4 mm
- net Net-(P9-Pad1): track 37.2 -> 0.00 mm
- net Net-(U1-Pad9): track 35.3 -> 0.51 mm
- net Net-(U1-Pad10): track 33.2 -> 0.00 mm
- net Net-(P7-Pad7): track 27.6 -> 0.51 mm
- net Net-(D3-Pad2): track 60.0 -> 34.6 mm
- net Net-(P1-Pad1): track 22.7 -> 45.9 mm
- net Net-(U1-Pad2): track 12.4 -> 0.00 mm
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
Commit message: Update Edukit
Parts:
- added R10: R, Resistors_SMD:R_1206, F.Cu at (109.2, 61.5)
- added R11: R0b, Resistors_SMD:R_2512, F.Cu at (133.3, 62.9)
- added R12: R0b, Resistors_SMD:R_2512, F.Cu at (118.7, 66.0)
- added R13: R, Resistors_SMD:R_1206, F.Cu at (153.0, 97.8)
- added R14: R0b, Resistors_SMD:R_2512, F.Cu at (110.7, 91.4)
- added R15: R0a, Resistors_SMD:R_1206, F.Cu at (155.2, 122.4)
- added R16: R0a, Resistors_SMD:R_1206, F.Cu at (144.0, 120.4)
- added R17: R0a, Resistors_SMD:R_2512, F.Cu at (166.9, 113.3)
- added R18: R0a, Resistors_SMD:R_1206, F.Cu at (166.1, 66.0)
- added R19: R0a, Resistors_SMD:R_1206, F.Cu at (140.2, 68.6)
- added R20: R0b, Resistors_SMD:R_2512, F.Cu at (155.7, 122.4)
- added R21: R0b, Resistors_SMD:R_2512, F.Cu at (117.5, 115.7)
- added R23: R0a, Resistors_SMD:R_1206, F.Cu at (145.7, 128.8)
- added R6: R, Resistors_SMD:R_1206, F.Cu at (125.7, 72.4)
- added R7: R, Resistors_SMD:R_1206, F.Cu at (143.3, 62.0)
- added R8: R, Resistors_SMD:R_1206, F.Cu at (138.7, 73.7)
- added R9: R0a, Resistors_SMD:R_1206, F.Cu at (135.1, 73.7)
- moved P10 0.90 mm to (143.5, 68.6), turned to 180 degrees
- moved P2 0.65 mm to (105.9, 97.0)
Connections:
- D1 pad 1: Net-(C1-Pad2) -> Net-(D1-Pad1)
- D2 pad 1: Net-(C1-Pad2) -> Net-(D1-Pad1)
- P7 pad 1: Net-(P11-Pad1) -> Net-(P7-Pad1)
- U1 pad 16: Net-(P11-Pad1) -> Net-(R16-Pad2)
- U1 pad 7: Net-(U1-Pad7) -> Net-(R15-Pad2)
- U1 pad 8: Net-(P11-Pad1) -> Net-(P7-Pad1)
- U2 pad 10: Net-(P11-Pad1) -> Net-(R11-Pad1)
- U2 pad 12: Net-(P10-Pad1) -> Net-(R9-Pad1)
- U2 pad 13: Net-(P9-Pad1) -> Net-(R8-Pad1)
- U2 pad 14: Net-(P11-Pad3) -> Net-(R6-Pad1)
- U2 pad 22: Net-(P8-Pad1) -> Net-(R7-Pad1)
- U2 pad 24: Net-(P7-Pad2) -> Net-(R21-Pad2)
- U2 pad 25: Net-(P3-Pad3) -> Net-(R14-Pad1)
- U2 pad 26: Net-(U1-Pad7) -> Net-(U1-Pad10)
- U2 pad 28: Net-(U1-Pad10) -> Net-(R15-Pad1)
- U2 pad 32: Net-(P10-Pad2) -> Net-(R10-Pad1)
- U4 pad 5: Net-(C1-Pad2) -> Net-(D1-Pad1)
Routing:
- net Net-(P10-Pad2): track 81.7 -> 207.8 mm
- net Net-(C1-Pad2): track 151.2 -> 36.3 mm
- net Net-(U1-Pad2): track 0.00 -> 82.7 mm
- net Net-(P7-Pad6): track 0.76 -> 78.5 mm
- net Net-(R15-Pad1): track 0.00 -> 68.3 mm
- net Net-(P7-Pad7): track 0.51 -> 57.0 mm
- net Net-(R17-Pad1): track 0.00 -> 56.4 mm
- net Net-(U1-Pad9): track 0.51 -> 53.1 mm
- net Net-(U1-Pad10): track 0.00 -> 48.3 mm
- net Net-(P7-Pad5): track 0.76 -> 48.6 mm
- net Net-(R10-Pad1): track 0.00 -> 46.7 mm
- net Net-(D3-Pad2): track 34.6 -> 79.1 mm
- net Net-(P9-Pad1): track 0.00 -> 39.6 mm
- net Net-(R7-Pad1): track 0.00 -> 36.7 mm
- net Net-(R21-Pad1): track 0.00 -> 33.8 mm
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