File: EduKit/EduKit.sch (KiCad schematic (older format))
At the start: 23 parts, among them P4 CONN_01X02, P7 CONN_01X02, U2 Arduino_Mini, U3 SPX2920U-3.3, U4 ESP8266

Commit message: Made PCB prototype
Parts:
- removed P7: CONN_01X02, Pin_Headers:Pin_Header_Straight_1x02, symbol CONN_01X02
- added D3: PowerLED, LEDs:LED-5MM, symbol LED
- added R5: R, Resistors_ThroughHole:Resistor_Horizontal_RM7mm, symbol R
- added U5: PowerButton, bugs:button, symbol button
- P1, P2: renamed from P?; value CONN_01X02 -> Wheel; footprint (none) -> Pin_Headers:Pin_Header_Straight_1x02
- P10: renamed from P?; value CONN_01X02 -> BlueLED; footprint (none) -> Pin_Headers:Pin_Header_Straight_1x02
- P11: renamed from P?; value CONN_01X03 -> IRReceiver; footprint (none) -> Pin_Headers:Pin_Header_Straight_1x03
- P3: renamed from P?; value CONN_01X04 -> Sonar; footprint (none) -> Pin_Headers:Pin_Header_Straight_1x04
- P4: value CONN_01X02 -> PowerPINs
- P5, P6: renamed from P?; value CONN_01X02 -> Headlight; footprint (none) -> Pin_Headers:Pin_Header_Straight_1x02
- P7: renamed from P?; value CONN_01X08 -> RCReader; footprint (none) -> Pin_Headers:Pin_Header_Straight_1x08
- P8: renamed from P?; value CONN_01X02 -> IRTransmitter; footprint (none) -> Pin_Headers:Pin_Header_Straight_1x02
- P9: renamed from P?; value CONN_01X02 -> RedLED; footprint (none) -> Pin_Headers:Pin_Header_Straight_1x02
- R1, R2, R3, R4: footprint w_pth_resistors:rc05_vert -> Resistors_ThroughHole:Resistor_Horizontal_RM7mm
- U1: renamed from U?; footprint (none) -> Housings_DIP:DIP-16_W7.62mm
Connections:
- net at P10.2 (P2), P11.2 (P2), P3.1 (P1)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: now also P8.2 (P2)
- net at U2.7 (RAW), U3.1 (VI): now also D3.2 (A), R5.2, U5.6 (C1)
- net at P4.1 (P1): now also U5.5 (B1)
- new net: D3.1 (K), R5.1
Changed lines of the file:
@@
 F 0 "R2" V 6800 3350 50  0000 C CNN
 F 1 "10k" V 6900 3350 50  0000 C CNN
-F 2 "w_pth_resistors:rc05_vert" V 6830 3350 50  0001 C CNN
+F 2 "Resistors_ThroughHole:Resistor_Horizontal_RM7mm" V 6830 3350 50  0001 C CNN
 F 3 "" H 6900 3350 50  0000 C CNN
 	1    6900 3350
@@
 F 0 "R3" V 7080 3350 50  0000 C CNN
 F 1 "10k" V 7000 3350 50  0000 C CNN
-F 2 "w_pth_resistors:rc05_vert" V 6930 3350 50  0001 C CNN
+F 2 "Resistors_ThroughHole:Resistor_Horizontal_RM7mm" V 6930 3350 50  0001 C CNN
 F 3 "" H 7000 3350 50  0000 C CNN
 	1    7000 3350
@@
 F 0 "R4" V 7180 5150 50  0000 C CNN
 F 1 "R" V 7100 5150 50  0000 C CNN
-F 2 "w_pth_resistors:rc05_vert" V 7030 5150 50  0001 C CNN
+F 2 "Resistors_ThroughHole:Resistor_Horizontal_RM7mm" V 7030 5150 50  0001 C CNN
 F 3 "" H 7100 5150 50  0000 C CNN
 	1    7100 5150
@@
 F 0 "R1" V 6880 5150 50  0000 C CNN
 F 1 "R" V 6800 5150 50  0000 C CNN
-F 2 "w_pth_resistors:rc05_vert" V 6730 5150 50  0001 C CNN
+F 2 "Resistors_ThroughHole:Resistor_Horizontal_RM7mm" V 6730 5150 50  0001 C CNN
 F 3 "" H 6800 5150 50  0000 C CNN
 	1    6800 5150
@@
 P 4800 1000
 F 0 "P4" H 4800 1150 50  0000 C CNN
-F 1 "CONN_01X02" V 4900 1000 50  0000 C CNN
+F 1 "PowerPINs" V 4900 1000 50  0000 C CNN
 F 2 "Pin_Headers:Pin_Header_Straight_1x02" H 4800 1000 50  0001 C CNN
 F 3 "" H 4800 1000 50  0000 C CNN
@@
 $EndComp
 $Comp
-L L293D U?
+L L293D U1
 U 1 1 587DD6FF
 P 2600 3650
-F 0 "U?" H 2900 4150 60  0000 C CNN
+F 0 "U1" H 2900 4150 60  0000 C CNN
 F 1 "L293D" H 2600 4150 60  0000 C CNN
-F 2 "" H 3150 3300 60  0000 C CNN
+F 2 "Housings_DIP:DIP-16_W7.62mm" H 3150 3300 60  0001 C CNN
 F 3 "" H 3150 3300 60  0000 C CNN
 	1    2600 3650
@@
 $EndComp
 $Comp
-L CONN_01X02 P?
+L CONN_01X02 P1
 U 1 1 587DE3C0
 P 1500 3550
-F 0 "P?" H 1500 3700 50  0000 C CNN
-F 1 "CONN_01X02" V 1600 3550 50  0000 C CNN
-F 2 "" H 1500 3550 50  0000 C CNN
+F 0 "P1" H 1500 3700 50  0000 C CNN
+F 1 "Wheel" V 1600 3550 50  0000 C CNN
+F 2 "Pin_Headers:Pin_Header_Straight_1x02" H 1500 3550 50  0001 C CNN
 F 3 "" H 1500 3550 50  0000 C CNN
 	1    1500 3550
@@
 $EndComp
 $Comp
-L CONN_01X02 P?
+L CONN_01X02 P2
 U 1 1 587DE533
 P 1500 4000
-F 0 "P?" H 1500 4150 50  0000 C CNN
-F 1 "CONN_01X02" V 1600 4000 50  0000 C CNN
-F 2 "" H 1500 4000 50  0000 C CNN
+F 0 "P2" H 1500 4150 50  0000 C CNN
+F 1 "Wheel" V 1600 4000 50  0000 C CNN
+F 2 "Pin_Headers:Pin_Header_Straight_1x02" H 1500 4000 50  0001 C CNN
 F 3 "" H 1500 4000 50  0000 C CNN
 	1    1500 4000
@@
 $EndComp
 $Comp
-L CONN_01X04 P?
+L CONN_01X04 P3
 U 1 1 587DEA8E
 P 1900 1700
-F 0 "P?" H 1900 1950 50  0000 C CNN
-F 1 "CONN_01X04" V 2000 1700 50  0000 C CNN
-F 2 "" H 1900 1700 50  0000 C CNN
+F 0 "P3" H 1900 1950 50  0000 C CNN
+F 1 "Sonar" V 2000 1700 50  0000 C CNN
+F 2 "Pin_Headers:Pin_Header_Straight_1x04" H 1900 1700 50  0001 C CNN
 F 3 "" H 1900 1700 50  0000 C CNN
 	1    1900 1700
@@
 $EndComp
 $Comp
-L CONN_01X02 P7
-U 1 1 5712384B
-P 4800 1350
-F 0 "P7" H 4800 1500 50  0000 C CNN
-F 1 "CONN_01X02" V 4900 1350 50  0000 C CNN
-F 2 "Pin_Headers:Pin_Header_Straight_1x02" H 4800 1350 50  0001 C CNN
-F 3 "" H 4800 1350 50  0000 C CNN
-	1    4800 1350
-	-1   0    0    1
-$EndComp
-$Comp
-L CONN_01X08 P?
+L CONN_01X08 P7
 U 1 1 587E510C
 P 4900 5500
-F 0 "P?" H 4900 5950 50  0000 C CNN
-F 1 "CONN_01X08" V 5000 5500 50  0000 C CNN
-F 2 "" H 4900 5500 50  0000 C CNN
+F 0 "P7" H 4900 5950 50  0000 C CNN
+F 1 "RCReader" V 5000 5500 50  0000 C CNN
+F 2 "Pin_Headers:Pin_Header_Straight_1x08" H 4900 5500 50  0001 C CNN
 F 3 "" H 4900 5500 50  0000 C CNN
 	1    4900 5500
@@
 $EndComp
 $Comp
-L CONN_01X02 P?
+L CONN_01X02 P6
 U 1 1 587E5CCD
 P 4450 6500
-F 0 "P?" H 4450 6650 50  0000 C CNN
-F 1 "CONN_01X02" V 4550 6500 50  0000 C CNN
-F 2 "" H 4450 6500 50  0000 C CNN
+F 0 "P6" H 4450 6650 50  0000 C CNN
+F 1 "Headlight" V 4550 6500 50  0000 C CNN
+F 2 "Pin_Headers:Pin_Header_Straight_1x02" H 4450 6500 50  0001 C CNN
 F 3 "" H 4450 6500 50  0000 C CNN
 	1    4450 6500
@@
 $EndComp
 $Comp
-L CONN_01X02 P?
+L CONN_01X02 P8
 U 1 1 587E5DE2
 P 4900 6250
-F 0 "P?" H 4900 6400 50  0000 C CNN
-F 1 "CONN_01X02" V 5000 6250 50  0000 C CNN
-F 2 "" H 4900 6250 50  0000 C CNN
+F 0 "P8" H 4900 6400 50  0000 C CNN
+F 1 "IRTransmitter" V 5000 6250 50  0000 C CNN
+F 2 "Pin_Headers:Pin_Header_Straight_1x02" H 4900 6250 50  0001 C CNN
 F 3 "" H 4900 6250 50  0000 C CNN
 	1    4900 6250
@@
 $EndComp
 $Comp
-L CONN_01X02 P?
+L CONN_01X02 P5
 U 1 1 587E5E3D
 P 4150 6500
-F 0 "P?" H 4150 6650 50  0000 C CNN
-F 1 "CONN_01X02" V 4250 6500 50  0000 C CNN
-F 2 "" H 4150 6500 50  0000 C CNN
+F 0 "P5" H 4150 6650 50  0000 C CNN
+F 1 "Headlight" V 4250 6500 50  0000 C CNN
+F 2 "Pin_Headers:Pin_Header_Straight_1x02" H 4150 6500 50  0001 C CNN
 F 3 "" H 4150 6500 50  0000 C CNN
 	1    4150 6500
@@
 $EndComp
 $Comp
-L CONN_01X02 P?
+L CONN_01X02 P10
 U 1 1 587E5F52
 P 5900 6250
-F 0 "P?" H 5900 6400 50  0000 C CNN
-F 1 "CONN_01X02" V 6000 6250 50  0000 C CNN
-F 2 "" H 5900 6250 50  0000 C CNN
+F 0 "P10" H 5900 6400 50  0000 C CNN
+F 1 "BlueLED" V 6000 6250 50  0000 C CNN
+F 2 "Pin_Headers:Pin_Header_Straight_1x02" H 5900 6250 50  0001 C CNN
 F 3 "" H 5900 6250 50  0000 C CNN
 	1    5900 6250
@@
 $EndComp
 $Comp
-L CONN_01X02 P?
+L CONN_01X02 P9
 U 1 1 587E5FE3
 P 5550 6250
-F 0 "P?" H 5550 6400 50  0000 C CNN
-F 1 "CONN_01X02" V 5650 6250 50  0000 C CNN
-F 2 "" H 5550 6250 50  0000 C CNN
+F 0 "P9" H 5550 6400 50  0000 C CNN
+F 1 "RedLED" V 5650 6250 50  0000 C CNN
+F 2 "Pin_Headers:Pin_Header_Straight_1x02" H 5550 6250 50  0001 C CNN
 F 3 "" H 5550 6250 50  0000 C CNN
 	1    5550 6250
@@
 $EndComp
 $Comp
-L CONN_01X03 P?
+L CONN_01X03 P11
 U 1 1 587E620C
 P 6250 6000
-F 0 "P?" H 6250 6200 50  0000 C CNN
-F 1 "CONN_01X03" V 6350 6000 50  0000 C CNN
-F 2 "" H 6250 6000 50  0000 C CNN
+F 0 "P11" H 6250 6200 50  0000 C CNN
+F 1 "IRReceiver" V 6350 6000 50  0000 C CNN
+F 2 "Pin_Headers:Pin_Header_Straight_1x03" H 6250 6000 50  0001 C CNN
 F 3 "" H 6250 6000 50  0000 C CNN
 	1    6250 6000
+	0    1    1    0
+$EndComp
+$Comp
+L button U5
+U 1 1 587F3CB4
+P 3500 1300
+F 0 "U5" V 3700 1250 60  0000 C CNN
+F 1 "PowerButton" V 3300 1200 60  0000 C CNN
+F 2 "bugs:button" H 3550 1300 60  0001 C CNN
+F 3 "" H 3550 1300 60  0000 C CNN
+	1    3500 1300
+	0    1    1    0
+$EndComp
+$Comp
+L LED D3
+U 1 1 587F401D
+P 4200 900
+F 0 "D3" H 4200 1000 50  0000 C CNN
+F 1 "PowerLED" H 4200 800 50  0000 C CNN
+F 2 "LEDs:LED-5MM" H 4200 900 50  0001 C CNN
+F 3 "" H 4200 900 50  0000 C CNN
+	1    4200 900
+	-1   0    0    1
+$EndComp
+$Comp
+L R R5
+U 1 1 587F4103
+P 4200 1100
+F 0 "R5" V 4280 1100 50  0000 C CNN
+F 1 "R" V 4200 1100 50  0000 C CNN
+F 2 "Resistors_ThroughHole:Resistor_Horizontal_RM7mm" V 4130 1100 50  0001 C CNN
+F 3 "" H 4200 1100 50  0000 C CNN
+	1    4200 1100
 	0    1    1    0
 $EndComp
@@
 Wire Wire Line
 	4950 4600 4800 4600
-Connection ~ 4850 6050
 Wire Wire Line
 	5500 6050 5500 5950
@@
 	6250 5800 4250 5800
 Connection ~ 4250 5800
+Wire Wire Line
+	4850 6050 4250 6050
+Connection ~ 4250 6050
+Wire Wire Line
+	3800 1400 5000 1400
+Wire Wire Line
+	5000 1300 3800 1300
+Wire Wire Line
+	4400 900  4400 1100
+Wire Wire Line
+	4400 1100 4350 1100
+Wire Wire Line
+	4050 1100 4050 1400
+Connection ~ 4050 1400
+Wire Wire Line
+	4000 900  4000 1400
+Connection ~ 4000 1400
 $EndSCHEMATC

Commit message: Jackalized a little
Parts:
- P10: value BlueLED -> Speaker
Changed lines of the file:
@@
 LIBS:valves
 LIBS:bugs
-LIBS:kidkit-cache
+LIBS:EduKit-cache
 EELAYER 25 0
 EELAYER END
@@
 $EndComp
 $Comp
-L CONN_01X02 P10
-U 1 1 587E5F52
-P 5900 6250
-F 0 "P10" H 5900 6400 50  0000 C CNN
-F 1 "BlueLED" V 6000 6250 50  0000 C CNN
-F 2 "Pin_Headers:Pin_Header_Straight_1x02" H 5900 6250 50  0001 C CNN
-F 3 "" H 5900 6250 50  0000 C CNN
-	1    5900 6250
-	0    1    1    0
-$EndComp
-$Comp
 L CONN_01X02 P9
 U 1 1 587E5FE3
@@
 	0    1    1    0
 $EndComp
+$Comp
+L CONN_01X02 P10
+U 1 1 5881EF5D
+P 5900 6250
+F 0 "P10" H 5900 6400 50  0000 C CNN
+F 1 "Speaker" V 6000 6250 50  0000 C CNN
+F 2 "Pin_Headers:Pin_Header_Straight_1x02" H 5900 6250 50  0001 C CNN
+F 3 "" H 5900 6250 50  0000 C CNN
+	1    5900 6250
+	0    1    1    0
+$EndComp
 Wire Wire Line
 	7250 3650 7100 3650
@@
 	5000 1050 5000 1300
 Wire Wire Line
-	5400 3350 6350 3350
-Wire Wire Line
 	5000 1400 5000 2000
 Wire Wire Line
@@
 Wire Wire Line
 	2000 4550 3450 4550
-Wire Wire Line
-	3450 4550 3450 2400
-Wire Wire Line
-	3450 3300 3100 3300
 Wire Wire Line
 	3900 3450 3900 2550
@@
 Connection ~ 4250 5950
 Wire Wire Line
-	5850 6050 5850 5900
-Wire Wire Line
-	5850 5900 4250 5900
-Connection ~ 4250 5900
-Wire Wire Line
 	5600 6050 5600 5600
 Wire Wire Line
@@
 Wire Wire Line
 	5800 3650 5400 3650
-Wire Wire Line
-	5950 6050 5950 3550
-Wire Wire Line
-	5950 3550 5400 3550
 Wire Wire Line
 	6150 5800 6150 3750
@@
 	4000 900  4000 1400
 Connection ~ 4000 1400
+Wire Wire Line
+	3450 4550 3450 2400
+Wire Wire Line
+	3100 3300 3450 3300
+Wire Wire Line
+	5400 3350 6350 3350
+Wire Wire Line
+	4250 5900 5850 5900
+Wire Wire Line
+	5850 5900 5850 6050
+Connection ~ 4250 5900
+Wire Wire Line
+	5950 6050 5950 3550
+Wire Wire Line
+	5950 3550 5400 3550
 $EndSCHEMATC

Commit message: Update Edukit
Parts:
- added R10, R13, R6, R7, R8: R, Resistors_SMD:R_1206, symbol R
- added R11, R12, R14, R20, R21: R0b, Resistors_SMD:R_2512, symbol R
- added R15, R16, R18, R19, R23, R9: R0a, Resistors_SMD:R_1206, symbol R
- added R17: R0a, Resistors_SMD:R_2512, symbol R
Connections:
- net at U2.12 (A2): now also R9.1; no longer P10.1 (P1)
- net at U2.13 (A1): now also R8.1; no longer P9.1 (P1)
- net at U2.14 (A0): now also R6.1; no longer P11.3 (P3)
- net at U2.22 (A5): now also R7.1; no longer P8.1 (P1)
- net at U2.24 (9): now also R21.2; no longer P7.2 (P2)
- net at U2.25 (8): now also R14.1; no longer P3.3 (P3)
- net at U2.26 (7): now also U1.10 (IN3); no longer U1.7 (IN2)
- net at U2.28 (5): now also R15.1; no longer U1.10 (IN3)
- net at P10.2 (P2), P11.2 (P2), P3.1 (P1)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: now also R10.2; no longer U2.32 (GND)
- net at C1.2, P4.2 (P2), U3.2 (GND): now also R13.1; no longer D1.1 (K), D2.1 (K), U4.5 (GND)
- new net: R11.1, R19.1, U2.10 (VCC)
- new net: R10.1, U2.32 (GND)
- new net: D1.1 (K), D2.1 (K), R13.2, U4.5 (GND)
- new net: R16.2, U1.16 (Vss)
- new net: R15.2, U1.7 (IN2)
- new net: P7.1 (P1), R17.2, R20.1, U1.8 (Vs)
- new net: P3.3 (P3), R12.2
- new net: P11.1 (P1), P3.4 (P4), R11.2
- new net: P7.2 (P2), R23.2
- new net: P8.1 (P1), R7.2
- new net: P9.1 (P1), R8.2
- new net: P11.3 (P3), R6.2
- new net: P10.1 (P1), R9.2
- new net: R12.1, R14.2
- new net: R16.1, R20.2
- new net: R17.1, R18.2
- new net: R18.1, R19.2
- new net: R21.1, R23.1
Other:
- moved on the sheet: P8
